File: layouts/default/default.kicad_pcb (KiCad board)
At the start: 2 copper layers, 69 parts

Commit message: layout floorplan complete
Parts:
- moved R12 354.8 mm to (111.3, 96.9)
- moved R9 352.2 mm to (104.3, 86.4)
- moved R14 341.1 mm to (126.3, 86.9)
- moved R11 334.9 mm to (108.3, 96.9)
- moved C9 318.4 mm to (111.3, 98.4)
- moved C10 314.1 mm to (110.8, 83.9)
- moved C11 303.3 mm to (123.8, 86.9)
- moved R6 298.5 mm to (124.3, 91.4), turned to 90 degrees
- moved R2 282.0 mm to (123.8, 83.4)
- moved C8 271.0 mm to (108.3, 98.4)
- moved R3 269.4 mm to (100.8, 89.9), turned to -90 degrees
- moved C7 247.9 mm to (104.3, 84.9)
- moved U1 244.9 mm to (110.8, 88.4), turned to -90 degrees
- moved U3 240.8 mm to (120.8, 88.4), turned to -90 degrees
- moved R5 229.5 mm to (99.3, 96.9), turned to -90 degrees
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Connections:
- net input_stage-P1INplus renamed P1INplus
- C1 pad 1: gain_stage-line -> gain_stage-line-1
- C11 pad 1: gain_stage-tap-1 -> anode
- C13 pad 1: hv -> hv-1
- C13 pad 2: gnd-1 -> gnd-3
- C15 pad 2: anode -> cathode
- C16 pad 2: gnd-1 -> gnd-3
- C17 pad 1: hv-1 -> hv
- C17 pad 2: gnd-1 -> gnd-3
- C18 pad 1: gnd-2 -> gnd
- C18 pad 2: gnd-1 -> gnd-3
- C19 pad 1: line-3 -> line
- C2 pad 1: line-3 -> line
- C2 pad 2: gain_stage-resistors_ifs[0] -> gain_stage-resistors_ifs[0]-1
- C21 pad 2: summing_opamp-output -> output-1
- C3 pad 1: gain_stage-resistors_ifs[0] -> gain_stage-resistors_ifs[0]-1
- C3 pad 2: gain_stage-net-1 -> gain_stage-net
- C4 pad 1: gain_stage-net-3 -> gain_stage-net-1
- C5 pad 1: gain_stage-net -> gain_stage-net-4
- C5 pad 2: line-1 -> line-2
- C6 pad 2: gain_stage-line-1 -> gain_stage-line
- C7 pad 1: gain_stage-line-1 -> gain_stage-line
- C7 pad 2: gain_stage-P1INplus -> gain_stage-resistors_ifs[0]
- C8 pad 1: gain_stage-net-4 -> gain_stage-net-3
- D1 pad 1: hv -> hv-1
- D1 pad 2: gnd-1 -> gnd-3
- D2 pad 1: anode -> cathode
- D2 pad 2: hv -> hv-1
- D3 pad 1: hv-1 -> hv
- D3 pad 2: anode -> cathode
- R1 pad 1: gain_stage-line-1 -> gain_stage-line
- R1 pad 2: gain_stage-line -> gain_stage-line-1
- R10 pad 2: gain_stage-net-4 -> gain_stage-net-3
- R11 pad 1: gain_stage-net-4 -> gain_stage-net-3
- R13 pad 2: gain_stage-tap-1 -> anode
- R14 pad 2: line-1 -> line-2
- R15 pad 1: gain_stage-P1INplus -> gain_stage-resistors_ifs[0]
- R17 pad 1: gain_stage-resistors_ifs[0] -> gain_stage-resistors_ifs[0]-1
- R2 pad 1: gain_stage-line -> gain_stage-line-1
- R2 pad 2: line-1 -> line-2
- R21 pad 2: gnd-1 -> gnd-3
- R22 pad 1: hv -> hv-1
- R23 pad 2: gnd -> gnd-2
- R24 pad 2: line -> line-1
- R26 pad 2: gnd-3 -> gnd-1
- R28 pad 1: line -> line-1
- R3 pad 1: line-3 -> line
- R3 pad 2: gain_stage-resistors_ifs[0] -> gain_stage-resistors_ifs[0]-1
- R30 pad 1: gnd-3 -> gnd-1
- R31 pad 2: summing_opamp-output -> output-1
- R34 pad 1: line-2 -> output-1
- R35 pad 1: line-2 -> output-1
- R4 pad 1: gain_stage-resistors_ifs[0] -> gain_stage-resistors_ifs[0]-1
- R5 pad 1: gain_stage-net-1 -> gain_stage-net
- R6 pad 2: gain_stage-net-3 -> gain_stage-net-1
- R7 pad 2: line-1 -> line-2
- R8 pad 2: gain_stage-net -> gain_stage-net-4
- R9 pad 1: gain_stage-line-1 -> gain_stage-line
- R9 pad 2: gain_stage-P1INplus -> gain_stage-resistors_ifs[0]
- U1 pad 3: gain_stage-P1INplus -> gain_stage-resistors_ifs[0]
- U1 pad 4: gnd-1 -> gnd-3
- U1 pad 8: hv -> hv-1
- U2 pad 1: gnd-1 -> gnd-3
- U2 pad 2: gain_stage-tap-1 -> anode
- U3 pad 1: gain_stage-tap-1 -> anode
- U3 pad 2: gnd-1 -> gnd-3
- U4 pad 4: gnd-1 -> gnd-3
- U4 pad 8: hv -> hv-1
- U5 pad 1: hv -> hv-1
- U5 pad 3: gnd-1 -> gnd-3
- U5 pad 5: gnd-2 -> gnd
- U5 pad 8: hv -> hv-1
- U6 pad 1: summing_opamp-output -> output-1
- U6 pad 4: gnd-2 -> gnd
- U6 pad 8: hv-1 -> hv
- U7 pad 4: gnd-2 -> gnd
- U7 pad 8: hv-1 -> hv
Other:
- board outline added: 100 x 50 mm
