File: layouts/default/default.kicad_pcb (KiCad board)
At the start: 2 copper layers, 100 x 50 mm, 69 parts

Commit message: fancy layout
Parts:
- added G***: LOGO, LOGO, F.Cu at (116.9, 88.4)
- C2, C7: value 68nF ±10% 16V X5R -> 68nF ±10% 16V X7R; footprint atopile:C0201-a4ec75 -> atopile:C0402-b3ef17
- C5: value 27nF ±10% 16V X7R -> 27nF ±10% 16V X5R; footprint atopile:C0402-b3ef17 -> atopile:C0201-a4ec75
- R14: value 47kΩ ±1% 62.5mW -> 47kΩ ±1% 100mW; footprint atopile:R0402-56259e -> atopile:R0603-ebcab9
- R36: value 4.7kΩ ±1% 100mW -> 4.7kΩ ±1% 62.5mW; footprint atopile:R0603-ebcab9 -> atopile:R0402-56259e
- R4: value 1.5kΩ ±1% 62.5mW -> 1.5kΩ ±1% 100mW; footprint atopile:R0402-56259e -> atopile:R0603-ebcab9
- moved C13 21.1 mm to (105.5, 108.0)
- moved D1 21.1 mm to (102.5, 107.9)
- moved C18 21.1 mm to (125.5, 111.7)
- moved R21 21.1 mm to (126.5, 106.6)
- moved R22 21.1 mm to (123.8, 105.6)
- moved C14 21.1 mm to (114.5, 111.0)
- moved C16 21.1 mm to (129.0, 107.7)
- moved C17 21.1 mm to (108.0, 109.5)
- moved D2 21.1 mm to (116.5, 104.0)
- moved D3 21.1 mm to (112.5, 107.5)
- moved U5 21.1 mm to (120.5, 109.0)
- moved C15 20.3 mm to (111.7, 110.8), turned to 90 degrees
- moved R23 11.8 mm to (144.5, 79.0), turned to 180 degrees
- moved R20 10.5 mm to (87.2, 80.5)
- moved C12 10.3 mm to (90.0, 80.5)
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Connections:
- net P1INplus renamed input_stage-P1INplus
- C1 pad 1: gain_stage-line-1 -> gain_stage-line
- C1 pad 2: gain_stage.ff1_low_pass-gnd -> gnd-3
- C10 pad 1: gain_stage-output -> output-1
- C10 pad 2: gain_stage-net-2 -> gain_stage-net-3
- C11 pad 1: anode -> gain_stage-tap
- C11 pad 2: gain_stage-tap -> gain_stage-tap-1
- C13 pad 1: hv-1 -> hv
- C13 pad 2: gnd-3 -> gnd-1
- C16 pad 2: gnd-3 -> gnd-1
- C17 pad 1: hv -> hv-1
- C17 pad 2: gnd-3 -> gnd-1
- C18 pad 1: gnd -> gnd-2
- C18 pad 2: gnd-3 -> gnd-1
- C19 pad 1: line -> output-1
- C2 pad 1: line -> output-1
- C2 pad 2: gain_stage-resistors_ifs[0]-1 -> gain_stage-resistors_ifs[0]
- C21 pad 1: summing_opamp-P1INminus -> P1INminus
- C21 pad 2: output-1 -> output-2
- C3 pad 1: gain_stage-resistors_ifs[0]-1 -> gain_stage-resistors_ifs[0]
- C3 pad 2: gain_stage-net -> gain_stage-net-5
- C4 pad 1: gain_stage-net-1 -> gain_stage-net-4
- C4 pad 2: gain_stage-tap -> gain_stage-tap-1
- C5 pad 1: gain_stage-net-4 -> gain_stage-net
- C5 pad 2: line-2 -> P1INminus
- C6 pad 1: gain_stage-output -> output-1
- C6 pad 2: gain_stage-line -> gain_stage-net-2
- C7 pad 1: gain_stage-line -> gain_stage-net-2
- C7 pad 2: gain_stage-resistors_ifs[0] -> gain_stage-P1INplus
- C8 pad 1: gain_stage-net-3 -> gain_stage-net-1
- C9 pad 2: gain_stage-output -> output-1
- D1 pad 1: hv-1 -> hv
- D1 pad 2: gnd-3 -> gnd-1
- D2 pad 2: hv-1 -> hv
- D3 pad 1: hv -> hv-1
- R1 pad 1: gain_stage-line -> output-1
- R1 pad 2: gain_stage-line-1 -> gain_stage-line
- R10 pad 2: gain_stage-net-3 -> gain_stage-net-1
- R11 pad 1: gain_stage-net-3 -> gain_stage-net-1
- R12 pad 2: gain_stage-output -> output-1
- R13 pad 1: gain_stage-net-2 -> gain_stage-net-3
- R13 pad 2: anode -> gain_stage-tap
- R14 pad 1: gain_stage-tap -> gain_stage-tap-1
- R14 pad 2: line-2 -> P1INminus
- R15 pad 1: gain_stage-resistors_ifs[0] -> gain_stage-P1INplus
- R17 pad 1: gain_stage-resistors_ifs[0]-1 -> gain_stage-resistors_ifs[0]
- R2 pad 1: gain_stage-line-1 -> gain_stage-line
- R2 pad 2: line-2 -> P1INminus
- R21 pad 2: gnd-3 -> gnd-1
- R22 pad 1: hv-1 -> hv
- R23 pad 2: gnd-2 -> gnd-3
- R24 pad 2: line-1 -> line
- R26 pad 2: gnd-1 -> gnd
- R28 pad 1: line-1 -> line
- R3 pad 1: line -> output-1
- R3 pad 2: gain_stage-resistors_ifs[0]-1 -> gain_stage-resistors_ifs[0]
- R30 pad 1: gnd-1 -> gnd
- R31 pad 1: summing_opamp-P1INminus -> P1INminus
- R31 pad 2: output-1 -> output-2
- R34 pad 1: output-1 -> output-2
- R35 pad 1: output-1 -> output-2
- R4 pad 1: gain_stage-resistors_ifs[0]-1 -> gain_stage-resistors_ifs[0]
- R5 pad 1: gain_stage-net -> gain_stage-net-5
- R6 pad 2: gain_stage-net-1 -> gain_stage-net-4
- R7 pad 2: line-2 -> P1INminus
- R8 pad 2: gain_stage-net-4 -> gain_stage-net
- R9 pad 1: gain_stage-line -> gain_stage-net-2
- R9 pad 2: gain_stage-resistors_ifs[0] -> gain_stage-P1INplus
- U1 pad 1: gain_stage-output -> output-1
- U1 pad 3: gain_stage-resistors_ifs[0] -> gain_stage-P1INplus
- U1 pad 4: gnd-3 -> gnd-1
- U1 pad 8: hv-1 -> hv
- U2 pad 1: gnd-3 -> gnd-1
- U2 pad 2: anode -> gain_stage-tap
- U3 pad 1: anode -> gain_stage-tap
- U3 pad 2: gnd-3 -> gnd-1
- U4 pad 1: input_stage.input_buffer_opamp-P1INminus -> output-1
- U4 pad 2: input_stage.input_buffer_opamp-P1INminus -> output-1
- U4 pad 4: gnd-3 -> gnd-1
- U4 pad 8: hv-1 -> hv
- U5 pad 1: hv-1 -> hv
- U5 pad 3: gnd-3 -> gnd-1
- U5 pad 5: gnd -> gnd-2
- U5 pad 8: hv-1 -> hv
- U6 pad 1: output-1 -> output-2
- U6 pad 2: summing_opamp-P1INminus -> P1INminus
- U6 pad 4: gnd -> gnd-2
- U6 pad 8: hv -> hv-1
- U7 pad 4: gnd -> gnd-2
- U7 pad 8: hv -> hv-1
Routing:
- net output-1: track 0.00 -> 131.4 mm, vias 0 -> 3
- net hv-2: track 0.00 -> 45.6 mm, vias 0 -> 1
- net hv: track 0.00 -> 31.1 mm, vias 0 -> 2
- net gain_stage-tap: track 0.00 -> 30.6 mm
- net output-2: track 0.00 -> 29.4 mm
- net gain_stage-wiper: track 0.00 -> 28.1 mm
- net gain_stage-P1INminus: track 0.00 -> 26.8 mm
- net P1INminus: track 0.00 -> 17.5 mm
- net tone_control-P1INminus: track 0.00 -> 16.6 mm
- net output: track 0.00 -> 15.6 mm, vias 0 -> 2
- net line: track 0.00 -> 14.0 mm
- net bypass-tap: track 0.00 -> 13.4 mm
- net tone_control-wiper: track 0.00 -> 13.3 mm
- net tone_control-resistors_ifs[0]: track 0.00 -> 12.9 mm
- net gain_stage-resistors_ifs[0]: track 0.00 -> 12.1 mm
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- added copper zone on F.Cu, net gnd-1
Other:
- board text added: "4V5"
- board text added: "9V"

Commit message: layout updates
Parts:
- moved R21 47.8 mm to (84.2, 84.2)
- moved C16 47.7 mm to (84.5, 90.5)
- moved R22 47.6 mm to (83.2, 80.5)
- moved D3 47.0 mm to (71.5, 84.5)
- moved U5 45.9 mm to (78.5, 90.5)
- moved C15 44.4 mm to (73.8, 87.8)
- moved C14 44.3 mm to (73.0, 95.5), turned to 90 degrees
- moved C18 44.3 mm to (84.5, 95.0)
- moved D2 42.7 mm to (78.5, 84.5)
- moved C17 42.2 mm to (69.7, 91.8)
- moved C13 41.3 mm to (69.0, 88.8), turned to 180 degrees
- moved D1 35.4 mm to (69.0, 96.5), turned to 180 degrees
- moved C12 7.36 mm to (97.0, 82.8)
- moved R20 7.36 mm to (94.2, 82.8)
- moved R28 5.42 mm to (160.5, 82.5), turned to 0 degrees
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Routing:
- net INPUT: track 5.05 -> 37.8 mm
- net output_stage-gnd: track 5.81 -> 28.9 mm
- net output: track 15.6 -> 35.9 mm, vias 2 -> 3
- net hv-1: track 4.91 -> 18.3 mm, vias 1 -> 2
- net output_stage-net: track 0.00 -> 12.8 mm
- net input_stage-P1INplus: track 4.27 -> 15.2 mm, vias 0 -> 2
- net line: track 14.0 -> 24.8 mm
- net gnd-1: track 8.10 -> 18.1 mm, vias 0 -> 2
- net gain_stage-line: track 0.00 -> 8.44 mm
- net gain_stage-net-2: track 8.79 -> 15.9 mm
- net output-1: track 131.4 -> 126.7 mm
- net CAPplus: track 7.43 -> 3.49 mm
- net P1INminus: track 17.5 -> 20.3 mm
- net CAPminus: track 2.66 -> 0.00 mm
- net gnd-2: track 2.36 -> 0.00 mm
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
Commit message: building on latest
Parts:
- removed G***: LOGO, LOGO
- C1, C21, C6: footprint atopile:C0603-bd72f6 -> YAGEO_CC0603KRX7R9BB104:C0603
- C10, C11: footprint atopile:C0402-b3ef17 -> Samsung_Electro_Mechanics_CL05A105KA5NQNC:C0402
- C12: footprint atopile:C0402-b3ef17 -> Samsung_Electro_Mechanics_CL05B104KO5NNNC:C0402
- C13, C16: footprint atopile:C1206-f0a137 -> Murata_Electronics_GRM31CR61E476ME44L:C1206
- C14, C15, C17, C18: footprint atopile:C0603-bd72f6 -> Samsung_Electro_Mechanics_CL10A105KB8NNNC:C0603
- C19: footprint atopile:C0603-bd72f6 -> Samsung_Electro_Mechanics_CL10A475KO8NNNC:C0603
- C2, C7: footprint atopile:C0402-b3ef17 -> YAGEO_CC0402KRX7R7BB683:C0402
- C20: value 4.7µF ±10% 50V X5R -> 4.7µF ±10% 50V X7R; footprint atopile:C0805-3b2e55 -> Samsung_Electro_Mechanics_CL31B475KBHNNNE:C1206
- C22: footprint atopile:C0402-b3ef17 -> FH_0402B392K500NT:C0402
- C3: footprint atopile:C0402-b3ef17 -> CCTC_TCC0402X5R394K160AT:C0402
- C4: footprint atopile:C0201-a4ec75 -> Murata_Electronics_GRM033R71E222KA12D:C0201
- C5: footprint atopile:C0201-a4ec75 -> VIIYONG_V273K0201X5R160NAT:C0201
- C8: footprint atopile:C0402-b3ef17 -> YAGEO_CC0603KRX7R7BB823:C0603
- C9: footprint atopile:C0201-a4ec75 -> Murata_Electronics_GRM0335C1E391JA01D:C0201
- D1: footprint atopile:SOD-123_L2.7-W1.6-LS3.7-RD-30fb4b -> MDD_Microdiode_Electronics_BZT52C12:SOD-123_L2.7-W1.6-LS3.7-RD
- D2, D3: footprint atopile:SMA_L4.3-W2.5-LS5.0-RD-e683d9 -> TWGMC_ES1D:SMA_L4.3-W2.5-LS5.0-RD
- R1, R13, R15, R16, R17, R18, R21, R22, R27, R28, R29, R30, R31, R32, R33, R5: footprint atopile:R0603-ebcab9 -> UNI_ROYAL_0603WAF1001T5E:R0603
- R10: footprint atopile:R0603-ebcab9 -> UNI_ROYAL_0603WAF2001T5E:R0603
- R11, R2: value 15kΩ ±1% 62.5mW -> 15kΩ ±1% 100mW; footprint atopile:R0402-56259e -> UNI_ROYAL_0603WAF1502T5E:R0603
- R12: footprint atopile:R0402-56259e -> YAGEO_AF0402FR_07422KL:R0402
- R14: value 47kΩ ±1% 100mW -> 47kΩ ±1% 62.5mW; footprint atopile:R0603-ebcab9 -> UNI_ROYAL_0402WGF4702TCE:R0402
- R19: footprint atopile:R0603-ebcab9 -> UNI_ROYAL_0603WAF1004T5E:R0603
- R20: footprint atopile:R0402-56259e -> UNI_ROYAL_0402WGF1002TCE:R0402
- R23, R26, R35, R37: footprint atopile:R0402-56259e -> UNI_ROYAL_0402WGF1003TCE:R0402
- R24, R25: footprint atopile:R0603-ebcab9 -> UNI_ROYAL_0603WAF5600T5E:R0603
- R3: footprint atopile:R0603-ebcab9 -> UNI_ROYAL_0603WAF5101T5E:R0603
- R34: value 1.8kΩ ±1% 62.5mW -> 1.8kΩ ±1% 100mW; footprint atopile:R0402-56259e -> UNI_ROYAL_0603WAF1801T5E:R0603
- R36: value 4.7kΩ ±1% 62.5mW -> 4.7kΩ ±1% 100mW; footprint atopile:R0402-56259e -> UNI_ROYAL_0603WAF4701T5E:R0603
- R4: footprint atopile:R0603-ebcab9 -> UNI_ROYAL_0603WAF1501T5E:R0603
- R6: footprint atopile:R0603-ebcab9 -> UNI_ROYAL_0603WAF2202T5E:R0603
- R7: value 27kΩ ±1% 100mW -> 27kΩ ±1% 62.5mW; footprint atopile:R0603-ebcab9 -> UNI_ROYAL_0402WGF2702TCE:R0402
- R8: footprint atopile:R0402-56259e -> RALEC_RTT021202FTH:R0402
- R9: footprint atopile:R0603-ebcab9 -> UNI_ROYAL_0603WAF1002T5E:R0603
- U1, U4, U6, U7: footprint atopile:SOIC-8_L5.0-W4.0-P1.27-LS6.0-BL-294f77 -> STMicroelectronics_TL072CDT:SOIC-8_L5.0-W4.0-P1.27-LS6.0-BL
- U2, U3: footprint atopile:SOD-123FL_L2.7-W1.8-LS3.8-RD-0c8348 -> STMicroelectronics_BAT41ZFILM:SOD-123FL_L2.7-W1.8-LS3.8-RD
- U5: footprint atopile:SOP-8_L4.9-W3.9-P1.27-LS6.0-BL-0d1ac6 -> XBLW_MAX1044ESA_XBLW:SOP-8_L4.9-W3.9-P1.27-LS6.0-BL
Connections:
- net gain_stage-P1INplus renamed gain_stage-resistors_ifs[0]-1
- net input_stage-P1INplus renamed P1INplus
- C10 pad 1: output-1 -> output
- C10 pad 2: gain_stage-net-3 -> gain_stage-net-4
- C11 pad 1: gain_stage-tap -> gain_stage-tap-1
- C11 pad 2: gain_stage-tap-1 -> gain_stage-tap
- C13 pad 1: hv -> hv-1
- C13 pad 2: gnd-1 -> gnd
- C16 pad 1: hv-2 -> hv
- C16 pad 2: gnd-1 -> gnd
- C17 pad 1: hv-1 -> hv-2
- C17 pad 2: gnd-1 -> gnd
- C18 pad 2: gnd-1 -> gnd
- C19 pad 1: output-1 -> output
- C2 pad 1: output-1 -> output
- C20 pad 1: output -> output-2
- C21 pad 2: output-2 -> output-1
- C4 pad 1: gain_stage-net-4 -> gain_stage-net
- C4 pad 2: gain_stage-tap-1 -> gain_stage-tap
- C5 pad 1: gain_stage-net -> gain_stage-net-3
- C6 pad 1: output-1 -> output
- C6 pad 2: gain_stage-net-2 -> gain_stage-net-1
- C7 pad 1: gain_stage-net-2 -> gain_stage-net-1
- C8 pad 1: gain_stage-net-1 -> gain_stage-net-2
- C9 pad 2: output-1 -> output
- D1 pad 1: hv -> hv-1
- D1 pad 2: gnd-1 -> gnd
- D2 pad 2: hv -> hv-1
- D3 pad 1: hv-1 -> hv-2
- R1 pad 1: output-1 -> output
- R10 pad 2: gain_stage-net-1 -> gain_stage-net-2
- R11 pad 1: gain_stage-net-1 -> gain_stage-net-2
- R12 pad 2: output-1 -> output
- R13 pad 1: gain_stage-net-3 -> gain_stage-net-4
- R13 pad 2: gain_stage-tap -> gain_stage-tap-1
- R14 pad 1: gain_stage-tap-1 -> gain_stage-tap
- R15 pad 2: hv-2 -> hv
- R16 pad 2: hv-2 -> hv
- R18 pad 1: hv-2 -> hv
- R19 pad 2: hv-2 -> hv
- R21 pad 1: hv-2 -> hv
- R21 pad 2: gnd-1 -> gnd
- R22 pad 1: hv -> hv-1
- R22 pad 2: hv-2 -> hv
- R26 pad 2: gnd -> gnd-1
- R3 pad 1: output-1 -> output
- R30 pad 1: gnd -> gnd-1
- R31 pad 2: output-2 -> output-1
- R34 pad 1: output-2 -> output-1
- R35 pad 1: output-2 -> output-1
- R36 pad 2: output -> output-2
- R37 pad 2: output -> output-2
- R4 pad 2: hv-2 -> hv
- R5 pad 2: hv-2 -> hv
- R6 pad 2: gain_stage-net-4 -> gain_stage-net
- R8 pad 2: gain_stage-net -> gain_stage-net-3
- R9 pad 1: gain_stage-net-2 -> gain_stage-net-1
- U1 pad 1: output-1 -> output
- U1 pad 4: gnd-1 -> gnd
- U1 pad 8: hv -> hv-1
- U2 pad 1: gnd-1 -> gnd
- U2 pad 2: gain_stage-tap -> gain_stage-tap-1
- U3 pad 1: gain_stage-tap -> gain_stage-tap-1
- U3 pad 2: gnd-1 -> gnd
- U4 pad 1: output-1 -> output
- U4 pad 2: output-1 -> output
- U4 pad 4: gnd-1 -> gnd
- U4 pad 8: hv -> hv-1
- U5 pad 1: hv -> hv-1
- U5 pad 3: gnd-1 -> gnd
- U5 pad 8: hv -> hv-1
- U6 pad 1: output-2 -> output-1
- U6 pad 3: hv-2 -> hv
- U6 pad 8: hv-1 -> hv-2
- U7 pad 1: output -> output-2
- U7 pad 3: hv-2 -> hv
- U7 pad 8: hv-1 -> hv-2
Routing:
- net output-1: track 126.7 -> 29.4 mm, vias 3 -> 0
- net output: track 35.9 -> 126.7 mm
- net gain_stage-tap-1: track 2.95 -> 30.6 mm
- net gain_stage-tap: track 30.6 -> 2.95 mm
- net hv-2: track 45.7 -> 18.3 mm, vias 1 -> 2
- net hv: track 29.1 -> 45.7 mm, vias 5 -> 1
- net gain_stage-net-2: track 15.9 -> 3.65 mm
- net gain_stage-net-1: track 3.65 -> 15.9 mm
- net hv-1: track 18.3 -> 29.1 mm, vias 2 -> 5
- net gnd-1: track 18.1 -> 7.79 mm, vias 2 -> 0
- net gnd: track 7.79 -> 18.1 mm, vias 0 -> 2
- net output-2: track 29.4 -> 35.9 mm, vias 0 -> 3
- net gain_stage-net-3: track 1.26 -> 2.32 mm
- net gain_stage-net-4: track 1.91 -> 1.26 mm
- added copper zone on F.Cu, net gnd
- removed copper zone on F.Cu, net gnd-1

Commit message: ripping through layout
Parts:
- added U10: , XBLW_MAX1044ESA_XBLW:SOP-8_L4.9-W3.9-P1.27-LS6.0-BL, F.Cu at (80.5, 89.0)
- added U11: , D6_Potentiometer:D6_Potentiometer, F.Cu at (120.0, 68.0)
- added U8: , D6_Potentiometer:D6_Potentiometer, F.Cu at (80.0, 68.0)
- added U9: , D6_Potentiometer:D6_Potentiometer, F.Cu at (160.0, 68.0)
- U5: footprint XBLW_MAX1044ESA_XBLW:SOP-8_L4.9-W3.9-P1.27-LS6.0-BL -> D6_Potentiometer:D6_Potentiometer
- moved U5 22.5 mm to (80.0, 68.0), turned to 0 degrees
- moved D1 7.95 mm to (76.8, 94.8)
- moved C14 4.61 mm to (74.0, 91.0), turned to 180 degrees
- moved C1 2.50 mm to (123.5, 82.5)
- moved C10 2.50 mm to (117.0, 82.0)
- moved C11 2.50 mm to (124.5, 84.5)
- moved C12 2.50 mm to (99.0, 81.3)
- moved C13 2.50 mm to (71.0, 87.3)
- moved C15 2.50 mm to (75.8, 86.2)
- moved C16 2.50 mm to (86.5, 89.0)
- moved C17 2.50 mm to (71.7, 90.3)
- moved C18 2.50 mm to (86.5, 93.5)
- moved C19 2.50 mm to (146.3, 76.0)
- moved C2 2.50 mm to (100.6, 86.4)
- moved C20 2.50 mm to (151.8, 80.5)
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Connections:
- net P1INplus renamed input_stage-P1INplus
- C1 pad 2: gnd-3 -> gnd-1
- C10 pad 2: gain_stage-net-4 -> gain_stage-net-5
- C11 pad 1: gain_stage-tap-1 -> gain_stage-tap
- C11 pad 2: gain_stage-tap -> gain_stage-tap-1
- C13 pad 1: hv-1 -> hv
- C14 pad 1: CAPminus -> CAPneg
- C14 pad 2: CAPplus -> CAPpos
- C15 pad 1: CAPplus -> CAPpos
- C16 pad 1: hv -> hv-1
- C18 pad 1: gnd-2 -> gnd-3
- C20 pad 1: output-2 -> output-1
- C21 pad 2: output-1 -> output-2
- C3 pad 2: gain_stage-net-5 -> gain_stage-net-2
- C4 pad 2: gain_stage-tap -> gain_stage-tap-1
- C5 pad 1: gain_stage-net-3 -> gain_stage-net-1
- C6 pad 2: gain_stage-net-1 -> gain_stage-net-3
- C7 pad 1: gain_stage-net-1 -> gain_stage-net-3
- C7 pad 2: gain_stage-resistors_ifs[0]-1 -> gain_stage-P1INplus
- C8 pad 1: gain_stage-net-2 -> gain_stage-net-4
- D1 pad 1: hv-1 -> hv
- D2 pad 2: hv-1 -> hv
- R10 pad 2: gain_stage-net-2 -> gain_stage-net-4
- R11 pad 1: gain_stage-net-2 -> gain_stage-net-4
- R13 pad 1: gain_stage-net-4 -> gain_stage-net-5
- R13 pad 2: gain_stage-tap-1 -> gain_stage-tap
- R14 pad 1: gain_stage-tap -> gain_stage-tap-1
- R15 pad 1: gain_stage-resistors_ifs[0]-1 -> gain_stage-P1INplus
- R15 pad 2: hv -> hv-1
- R16 pad 2: hv -> hv-1
- R18 pad 1: hv -> hv-1
- R19 pad 2: hv -> hv-1
- R20 pad 1: INPUT-1 -> INPUT
- R21 pad 1: hv -> hv-1
- R22 pad 1: hv-1 -> hv
- R22 pad 2: hv -> hv-1
- R23 pad 2: gnd-3 -> gnd-1
- R26 pad 1: INPUT -> INPUT-1
- R26 pad 2: gnd-1 -> gnd-2
- R27 pad 1: INPUT -> INPUT-1
- R28 pad 2: INPUT -> INPUT-1
- R30 pad 1: gnd-1 -> gnd-2
- R31 pad 2: output-1 -> output-2
- R34 pad 1: output-1 -> output-2
- R35 pad 1: output-1 -> output-2
- R36 pad 2: output-2 -> output-1
- R37 pad 2: output-2 -> output-1
- R4 pad 2: hv -> hv-1
- R5 pad 1: gain_stage-net-5 -> gain_stage-net-2
- R5 pad 2: hv -> hv-1
- R8 pad 2: gain_stage-net-3 -> gain_stage-net-1
- R9 pad 1: gain_stage-net-1 -> gain_stage-net-3
- R9 pad 2: gain_stage-resistors_ifs[0]-1 -> gain_stage-P1INplus
- U1 pad 3: gain_stage-resistors_ifs[0]-1 -> gain_stage-P1INplus
- U1 pad 8: hv-1 -> hv
- U2 pad 2: gain_stage-tap-1 -> gain_stage-tap
- U3 pad 1: gain_stage-tap-1 -> gain_stage-tap
- U4 pad 8: hv-1 -> hv
- U5 pad 1: hv-1 -> gain_stage-P1INplus
- U5 pad 2: CAPplus -> hv-1
- U5 pad 3: gnd -> gain_stage-resistors_ifs[1]
- U6 pad 1: output-1 -> output-2
- U6 pad 3: hv -> hv-1
- U6 pad 4: gnd-2 -> gnd-3
- U7 pad 1: output-2 -> output-1
- U7 pad 3: hv -> hv-1
- U7 pad 4: gnd-2 -> gnd-3
Routing:
- net INPUT-1: track 0.87 -> 37.8 mm, vias 1 -> 0
- net gain_stage-tap-1: track 30.6 -> 2.95 mm
- net gain_stage-tap: track 2.95 -> 30.6 mm
- net hv-1: track 29.1 -> 45.7 mm, vias 5 -> 1
- net gain_stage-net-3: track 2.32 -> 15.9 mm
- net gain_stage-net-1: track 15.9 -> 2.32 mm
- net hv: track 45.7 -> 32.4 mm, vias 1 -> 5
- net INPUT: track 37.8 -> 25.2 mm, vias 0 -> 2
- net gain_stage-resistors_ifs[0]-1: track 10.8 -> 0.00 mm
- net gain_stage-P1INplus: track 0.00 -> 10.8 mm
- net gnd-2: track 0.00 -> 7.79 mm
- net gnd-1: track 7.79 -> 0.00 mm
- net output-2: track 35.9 -> 29.4 mm, vias 3 -> 0
- net output-1: track 29.4 -> 35.9 mm, vias 0 -> 3
- net CAPpos: track 0.00 -> 3.49 mm
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- added copper zone on F.Cu, net INPUT
Other:
- board size 100 x 50 mm -> 104 x 36 mm
- board text added: "INPUT GND"
- board text added: "INPUT SIGNAL"
- board text added: "OUTPUT GND"
- board text added: "OUTPUT SIGNAL"

Commit message: fighting off the rats
Parts:
- added R38: 10kΩ ±1% 100mW, UNI_ROYAL_0603WAF1002T5E:R0603, F.Cu at (0.00, 0.00)
- C20: footprint Samsung_Electro_Mechanics_CL31B475KBHNNNE:C1206 -> FH_1206B475K500NT:C1206
- R1, R15, R16, R17, R18, R21, R22, R27, R28, R29, R30, R31, R32, R33: value 1kΩ ±1% 100mW -> 10kΩ ±1% 100mW; footprint UNI_ROYAL_0603WAF1001T5E:R0603 -> UNI_ROYAL_0603WAF1002T5E:R0603
- U5: moved to B.Cu
- moved R15 0.25 mm to (107.1, 84.0)
- moved R22 0.25 mm to (85.0, 79.0)
- turned U5 to 180 degrees
Routing:
- net hv-1: track 45.7 -> 147.2 mm, vias 1 -> 10
- net hv-2: track 18.3 -> 118.2 mm, vias 2 -> 4
- net gnd-3: track 0.00 -> 86.1 mm, vias 0 -> 3
- net gain_stage-wiper: track 26.0 -> 88.0 mm, vias 0 -> 3
- net gain_stage-resistors_ifs[1]: track 1.50 -> 61.2 mm, vias 0 -> 2
- net hv: track 32.4 -> 82.6 mm, vias 5 -> 6
- net tone_control-resistors_ifs[1]: track 11.0 -> 60.3 mm, vias 0 -> 2
- net gain_stage-P1INplus: track 10.8 -> 53.4 mm, vias 0 -> 2
- net tone_control-resistors_ifs[0]: track 12.3 -> 54.6 mm, vias 0 -> 2
- net tone_control-wiper: track 15.2 -> 57.1 mm, vias 0 -> 2
- net gain_stage-resistors_ifs[0]: track 13.6 -> 52.3 mm, vias 0 -> 2
- net gnd-1: track 0.00 -> 27.8 mm, vias 0 -> 2
- net gnd-2: track 7.79 -> 31.2 mm, vias 0 -> 2
- net output_stage-resistors_ifs[0]: track 3.12 -> 23.7 mm, vias 0 -> 2
- net output_stage-gnd: track 28.9 -> 43.8 mm, vias 0 -> 2
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- added copper zone on F.Cu, net INPUT-1
- added copper zone on B.Cu, net gnd
- added copper zone on F.Cu, net gnd-2

Commit message: layout nearly complete
Parts:
- removed R38: 10kΩ ±1% 100mW, UNI_ROYAL_0603WAF1002T5E:R0603
Routing:
- net gain_stage-wiper: track 88.0 -> 93.0 mm, vias 3 -> 4
- net gnd: track 24.0 -> 28.4 mm, vias 21 -> 23
- net hv-1: track 147.2 -> 149.5 mm, vias 10 -> 11
- net hv: track 82.6 -> 84.7 mm, vias 6 -> 7
- net gnd-3: track 86.1 -> 88.1 mm, vias 3 -> 4
- net hv-2: track 118.2 -> 120.1 mm
- net gain_stage-resistors_ifs[0]: track 52.3 -> 53.6 mm
Other:
- board text added: "-9V"
- board text added: "16V"
- board text added: "9VBatt"
- board text added: "GND"
- board text removed: "9V"
